File: LockNFC_PCB/LockNFC.brd (EAGLE design)
At the start: 60 x 100 mm, 58 parts, among them J1 TC2030-MSP430-NO-UART-NL, Q3 13.56MHz

Commit message: Valid code/tag then choose a door (1 or 2) to open
Parts:
- C46: value 27p -> 68pF
- C47: value 27p -> 15pF
- C48: value 68p -> 100pF
- C49: value 10p -> 47pF
